File: jfet-radio/jfet-radio.kicad_sch (KiCad schematic)
At the start: 8 parts, among them Q1 Q_NJFET_DGS, Q2 Q_NJFET_DGS

Commit message: add feature
Parts:
- V2: Spice_Model dc 0 -> ac 1v 1k
Changed lines of the file:
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@@
       (effects (font (size 1.27 1.27)) (justify left) hide)
     )
-    (property "Spice_Model" "dc 0" (id 6) (at 105.5997 80.01 90))
+    (property "Spice_Model" "ac 1v 1k" (id 6) (at 105.5997 80.01 90))
     (pin "1")
     (pin "2")
